Commit message: SBAI upload

File: src/kobuki_ros/kobuki_description/model/kobuki_sim.gazebo.xacro (robot description, xacro)
@@ -8,16 +8,10 @@
       </hardware>
       <joint name="left_wheel_joint">
-        <command_interface name="velocity">
-          <param name="min">-1</param>
-          <param name="max">1</param>
-        </command_interface>
+        <command_interface name="velocity"/>
         <state_interface name="position"/>
         <state_interface name="velocity"/>
       </joint>
       <joint name="right_wheel_joint">
-        <command_interface name="velocity">
-          <param name="min">-1</param>
-          <param name="max">1</param>
-        </command_interface>
+        <command_interface name="velocity"/>
         <state_interface name="position"/>
         <state_interface name="velocity"/>

File: src/kobuki_ros/kobuki_description/model/kobuki_sim.xacro (robot description, xacro)
@@ -16,4 +16,9 @@
       <origin xyz="0 0 0.16438"/>
     </xacro:kobuki_base1>
+    <!-- <joint name="base_footprint_joint" type="fixed">
+      <parent link="odom"/>
+      <child link="base_footprint"/>
+      <origin xyz="0 0 0" rpy="0 0 0"/>
+    </joint> -->
     <xacro:kobuki_base2 parent="base_link">
       <origin xyz="0.0 0.0 0.154"/>

File: src/kobuki_ros/kobuki_description/model/wheels/kobuki_wheels.gazebo.xacro (robot description, xacro)
@@ -8,5 +8,5 @@
         <kd>100.0</kd>
         <minDepth>0.001</minDepth>
-        <maxVel>1.0</maxVel>
+        <maxVel>10.0</maxVel>
         <!-- <material>Gazebo/Yellow</material> -->
     </gazebo>

File: src/kobuki_ros/kobuki_description/model/wheels/kobuki_wheels.xacro (robot description, xacro)
@@ -7,5 +7,5 @@
             <parent link="${parent}"/>
             <child link="${prefix}_wheel_link"/>
-            <limit effort="50000" velocity="10"/>
+            <limit effort="50000" velocity="20"/>
             <dynamics damping="1.0" friction="1.0"/>
             <axis xyz="0 0 1"/>
