Commit message: Adding files for kobuki with D1-550 arm (Unitree)

File: src/kobuki_ros/kobuki_description/model/D1/D1.urdf.xacro (robot description, xacro)
@@ -64,5 +64,5 @@
         </link>
         <joint name="D1_joint_2" type="revolute"> <!-- type="revolute"> -->
-            <origin xyz="0 -0.0276 0.0578" rpy="0 0 0"/>
+            <origin xyz="0 -0.0276 0.0578" rpy="0 -0.90 0"/>
             <parent link="D1_link_1"/>
             <child link="D1_link_2"/>
@@ -94,5 +94,5 @@
         <joint
             name="D1_joint_3" type="revolute"> <!-- type="revolute"> -->
-            <origin xyz="0 -0.0004 0.27" rpy="0 0 0"/>
+            <origin xyz="0 -0.0004 0.27" rpy="0 1.57 0"/>
             <parent link="D1_link_2"/>
             <child link="D1_link_3"/>

File: src/kobuki_ros/kobuki_description/model/kobuki_d1_sim.gazebo.xacro (robot description, xacro)
@@ -17,4 +17,34 @@
         <state_interface name="velocity"/>
       </joint>
+      <joint name="D1_joint_1">
+        <command_interface name="position"/>
+        <state_interface name="position"/>
+        <state_interface name="velocity"/>
+      </joint>
+      <joint name="D1_joint_2">
+        <command_interface name="position"/>
+        <state_interface name="position"/>
+        <state_interface name="velocity"/>
+      </joint>
+      <joint name="D1_joint_3">
+        <command_interface name="position"/>
+        <state_interface name="position"/>
+        <state_interface name="velocity"/>
+      </joint>
+      <joint name="D1_joint_4">
+        <command_interface name="position"/>
+        <state_interface name="position"/>
+        <state_interface name="velocity"/>
+      </joint>
+      <joint name="D1_joint_5">
+        <command_interface name="position"/>
+        <state_interface name="position"/>
+        <state_interface name="velocity"/>
+      </joint>
+      <joint name="D1_joint_6">
+        <command_interface name="position"/>
+        <state_interface name="position"/>
+        <state_interface name="velocity"/>
+      </joint>
     </ros2_control>
     <gazebo>
@@ -29,5 +59,5 @@
           <namespace>$(arg namespace)</namespace>
         </ros>
-        <parameters>$(find kobuki_description)/config/kobuki_control.yaml</parameters>
+        <parameters>$(find kobuki_description)/config/kobuki_d1_control.yaml</parameters>
       </plugin>
     </gazebo>

File: src/kobuki_ros/kobuki_description/model/kobuki_d1_sim.xacro (robot description, xacro)
@@ -3,5 +3,5 @@
 <robot name="kobuki" xmlns:xacro="http://www.ros.org/wiki/xacro">
     <xacro:include filename="$(find kobuki_description)/model/common_properties.urdf.xacro" />
-    <xacro:include filename="$(find kobuki_description)/model/kobuki_sim.gazebo.xacro"/>
+    <xacro:include filename="$(find kobuki_description)/model/kobuki_d1_sim.gazebo.xacro"/>
     <xacro:include filename="$(find kobuki_description)/model/parts/kobuki_base.xacro"/>
     <xacro:include filename="$(find kobuki_description)/model/wheels/kobuki_wheels.xacro"/>
@@ -9,4 +9,5 @@
     <xacro:include filename="$(find kobuki_description)/model/sensors/imu/kobuki_imu.xacro"/>
     <xacro:include filename="$(find kobuki_description)/model/camera/kobuki_camera.xacro"/>
+    <xacro:include filename="$(find kobuki_description)/model/D1/D1.urdf.xacro"/>
     <link name="base_footprint"> </link>
                                                                           <!-- KOBUKI BASE -->
@@ -60,8 +61,8 @@
     <xacro:caster_gazebo prefix="back"/>
                                                                           <!-- KOBUKI LIDAR -->
-    <xacro:kobuki_lidar parent="base2_link">
+    <!-- <xacro:kobuki_lidar parent="base2_link">
         <origin xyz="0.0 0.0 0.030" rpy="0 0 0"/>
     </xacro:kobuki_lidar>
-    <xacro:lidar_gazebo/>
+    <xacro:lidar_gazebo/> -->
                                                                           <!-- KOBUKI IMU -->
     <xacro:kobuki_imu parent="base_link">
@@ -77,4 +78,9 @@
     <xacro:depth_camera_gazebo/> -->
     <xacro:rgbd_camera/>
+                                                                          <!-- D1 ARM -->
+    <xacro:D1_robot parent="base2_link">
+        <origin xyz="0.0 0.0 0.0010" rpy="0 0 0"/>
+    </xacro:D1_robot>
+    <xacro:D1_gazebo/>
                                                                           <!-- CONTROL -->
     <xacro:control_gazebo/>
