Commit message: 14-07-25

File: src/kobuki_ros/kobuki_description/model/camera/kobuki_camera.gazebo.xacro (robot description, xacro)
@@ -4,15 +4,20 @@
     <gazebo reference="camera_link">
         <sensor name="rgb_camera" type="camera">
+            <pose relative_to='camera_link'> 0 0 0 0 -0.174532925 0 </pose>
+            <gz_frame_id>camera_link</gz_frame_id>
+            <topic>rgb_camera</topic>
+            <always_on>1</always_on>
+            <update_rate>15</update_rate>
+            <visualize>true</visualize>
             <camera name="RGB_Camera">
-                <updateRate>30.0</updateRate>
-                <horizontal_fov>1.3962634</horizontal_fov>
+                <horizontal_fov>1.134464014</horizontal_fov>
                 <image>
-                    <width>640</width>
-                    <height>480</height>
+                    <width>320</width>
+                    <height>240</height>
                     <format>R8G8B8</format>
                 </image>
                 <clip>
-                    <near>0.3</near>
-                    <far>300</far>
+                    <near>0.1</near>
+                    <far>5</far>
                 </clip>
             </camera>
@@ -24,15 +29,18 @@
     <gazebo reference="camera_link">
         <sensor name="depth_camera" type="depth">
+            <pose relative_to='camera_link'> 0 0 0 0 -0.174532925 0 </pose>
+            <gz_frame_id>camera_link</gz_frame_id>
+            <topic>depth_camera</topic>
             <camera name="Depth_Camera">
-                <updateRate>30</updateRate>
-                <horizontal_fov>1.3962634</horizontal_fov>
+                <updateRate>15</updateRate>
+                <horizontal_fov>1.134464014</horizontal_fov>
                 <image>
-                    <width>640</width>
-                    <height>480</height>
+                    <width>320</width>
+                    <height>240</height>
                     <format>R8G8B8</format>
                 </image>
                 <clip>
-                    <near>0.3</near>
-                    <far>300</far>
+                    <near>0.1</near>
+                    <far>5</far>
                 </clip>
             </camera>
@@ -41,3 +49,26 @@
     </gazebo>
   </xacro:macro>
+  <xacro:macro name="rgbd_camera">
+    <gazebo reference="camera_link">
+        <sensor name="rgbd_camera" type="rgbd_camera">
+            <!-- <pose relative_to='camera_link'> 0 0 0 0 -0.174532925 0 </pose> -->
+            <pose relative_to='camera_link'> 0 0 0 0 0 0 </pose>
+            <gz_frame_id>camera_link</gz_frame_id>
+            <topic>rgbd_camera</topic>
+            <always_on>1</always_on>
+            <update_rate>2</update_rate>
+            <camera>
+                <horizontal_fov>1.134464014</horizontal_fov>
+                <image>
+                    <width>320</width>
+                    <height>240</height>
+                </image>
+                <clip>
+                    <near>0.1</near>
+                    <far>5</far>
+                </clip>
+            </camera>
+        </sensor>
+    </gazebo>
+  </xacro:macro>
 </robot>

File: src/kobuki_ros/kobuki_description/model/camera/kobuki_camera.xacro (robot description, xacro)
@@ -7,23 +7,22 @@
             <parent link="${parent}"/>
             <child link="camera_link"/>
-            <!-- <axis xyz="1 0 0"/> -->
         </joint>
         <link name="camera_link">
             <visual>
-                <origin xyz="0.16 -0.0 0.0" rpy="${-PI/2} 0 ${-PI/2}"/>
                 <geometry>
-                    <mesh filename="file://$(find kobuki_description)/meshes/stl/d415s.stl" />
-                    <!-- <box size="0.1 0.02 0.02"/> -->
+                    <mesh filename="file://$(find kobuki_description)/meshes/stl/d415s_rotated.stl" />
                 </geometry>
+                <xacro:insert_block name="material_light_grey"/>
+                <origin xyz="0 0 0" rpy="0 ${PI/2} 0"/>
             </visual>
             <collision>
                 <geometry>
-                    <mesh filename="file://$(find kobuki_description)/meshes/stl/d415s.stl" />
+                    <mesh filename="file://$(find kobuki_description)/meshes/stl/d415s_rotated.stl" />
                 </geometry>
-                <origin xyz="0.16 -0.0 0.0" rpy="${-PI/2} 0 ${-PI/2}"/>
+                <origin xyz="0 0 0" rpy="0 ${PI/2} 0"/>
             </collision>
             <inertial>
                 <origin xyz="0 0 0.0"/>
-                <mass value="0.072"/>
+                <mass value="0.064"/>
                 <inertia ixx="0.003881243" ixy="0" ixz="0" iyy="0.000498940" iyz="0" izz="0.003879257" />
             </inertial>

File: src/kobuki_ros/kobuki_description/model/common_properties.urdf.xacro (robot description, xacro)
@@ -5,4 +5,5 @@
 <robot name="xacro_properties" xmlns:xacro="http://ros.org/wiki/xacro">
   <xacro:property name="PI" value="3.1415926535897931" />
+  <xacro:property name="max_vel" value="30" /> <!-- 7m/s, 1.91rad/s -->
   <xacro:property name="material_white">
     <material name="white">

File: src/kobuki_ros/kobuki_description/model/kobuki_sim.gazebo.xacro (robot description, xacro)
@@ -17,6 +17,41 @@
         <state_interface name="velocity"/>
       </joint>
+      <joint name="D1_joint_1">
+        <command_interface name="position"/>
+        <state_interface name="position"/>
+        <state_interface name="velocity"/>
+      </joint>
+      <joint name="D1_joint_2">
+        <command_interface name="position"/>
+        <state_interface name="position"/>
+        <state_interface name="velocity"/>
+      </joint>
+      <joint name="D1_joint_3">
+        <command_interface name="position"/>
+        <state_interface name="position"/>
+        <state_interface name="velocity"/>
+      </joint>
+      <joint name="D1_joint_4">
+        <command_interface name="position"/>
+        <state_interface name="position"/>
+        <state_interface name="velocity"/>
+      </joint>
+      <joint name="D1_joint_5">
+        <command_interface name="position"/>
+        <state_interface name="position"/>
+        <state_interface name="velocity"/>
+      </joint>
+      <joint name="D1_joint_6">
+        <command_interface name="position"/>
+        <state_interface name="position"/>
+        <state_interface name="velocity"/>
+      </joint>
     </ros2_control>
     <gazebo>
+    <!-- Sensors plugin -->
+      <plugin filename="gz-sim-sensors-system" name="gz::sim::systems::Sensors">
+          <render_engine>ogre2</render_engine>
+      </plugin>
+      <plugin filename="gz-sim-imu-system" name="gz::sim::systems::Imu"> </plugin>
     <!-- Joint state publisher -->
       <plugin filename="gz_ros2_control-system" name="gz_ros2_control::GazeboSimROS2ControlPlugin">

File: src/kobuki_ros/kobuki_description/model/kobuki_sim.xacro (robot description, xacro)
@@ -9,71 +9,79 @@
     <xacro:include filename="$(find kobuki_description)/model/sensors/imu/kobuki_imu.xacro"/>
     <xacro:include filename="$(find kobuki_description)/model/camera/kobuki_camera.xacro"/>
-    <!-- <link name="base_footprint"/> -->
-    <link name="base_footprint">
-    </link>
+    <xacro:include filename="$(find kobuki_description)/model/D1/D1.urdf.xacro"/>
+    <link name="base_footprint"> </link>
+                                                                          <!-- KOBUKI BASE -->
     <xacro:kobuki_base1 parent="base_footprint">
-      <!-- <origin xyz="0 0 0.16438"/> -->
-      <origin xyz="0 0 0.16438"/>
+      <origin xyz="0 0 0.352"/>
     </xacro:kobuki_base1>
-    <!-- <joint name="base_footprint_joint" type="fixed">
-      <parent link="odom"/>
-      <child link="base_footprint"/>
-      <origin xyz="0 0 0" rpy="0 0 0"/>
-    </joint> -->
+    <xacro:base1_gazebo/>
+                                                                          <!-- KOBUKI BASE 2 -->
     <xacro:kobuki_base2 parent="base_link">
-      <origin xyz="0.0 0.0 0.154"/>
+      <origin xyz="0.0 0.0 0.10201"/>
     </xacro:kobuki_base2>
+    <xacro:base2_gazebo/>
+                                                                          <!-- KOBUKI PC -->
     <xacro:kobuki_pc parent="base_link">
-        <origin xyz="0.045 -0.0 0.121" rpy="0 0 ${PI}"/>
+        <origin xyz="0.045 0.0 0.06901"/>
     </xacro:kobuki_pc>
+    <xacro:pc_gazebo/>
+                                                                          <!-- KOBUKI HEX -->
     <xacro:kobuki_hex parent="base_link" prefix="back_left">
-      <origin xyz="-0.055 -0.12 0.12038"/>
+      <origin xyz="-0.055 -0.12 0.06901"/>
     </xacro:kobuki_hex>
+    <xacro:hex_gazebo prefix="back_left"/>
     <xacro:kobuki_hex parent="base_link" prefix="back_right">
-      <origin xyz="-0.055 0.12 0.12038"/>
+      <origin xyz="-0.055 0.12 0.06901"/>
     </xacro:kobuki_hex>
+    <xacro:hex_gazebo prefix="back_right"/>
     <xacro:kobuki_hex parent="base_link" prefix="front_left">
-      <origin xyz="0.055 -0.12 0.12038"/>
+      <origin xyz="0.055 -0.12 0.06901"/>
     </xacro:kobuki_hex>
+    <xacro:hex_gazebo prefix="front_left"/>
     <xacro:kobuki_hex parent="base_link" prefix="front_right">w
-      <origin xyz="0.055 0.12 0.12038"/>
+      <origin xyz="0.055 0.12 0.06901"/>
     </xacro:kobuki_hex>
+    <xacro:hex_gazebo prefix="front_right"/>
+                                                                          <!-- KOBUKI WHEELS -->
     <xacro:kobuki_wheel parent="base_link" prefix="right">
-        <origin xyz="0.00 -${0.23/2} 0.0250" rpy="${-PI/2} 0 0"/>
+        <origin xyz="0.00 -${0.23/2} -0.02699" rpy="${-PI/2} 0 0"/>
     </xacro:kobuki_wheel>
+    <xacro:wheel_gazebo prefix="right"/>
     <xacro:kobuki_wheel parent="base_link" prefix="left">
-        <origin xyz="0.00 ${0.23/2} 0.0250" rpy="${-PI/2} 0 0"/>
+        <origin xyz="0.00 ${0.23/2} -0.02699" rpy="${-PI/2} 0 0"/>
     </xacro:kobuki_wheel>
+    <xacro:wheel_gazebo prefix="left"/>
     <xacro:kobuki_caster parent="base_link" prefix="front">
-        <origin xyz="0.115 0.0 0.007" rpy="${-PI/2} 0 0"/>
+        <origin xyz="0.115 0.0 -0.04499" rpy="${-PI/2} 0 0"/>
     </xacro:kobuki_caster>
+    <xacro:caster_gazebo prefix="front"/>
     <xacro:kobuki_caster parent="base_link" prefix="back">
-        <origin xyz="-0.005 0.0 0.009" rpy="${-PI/2} 0 0"/>
+        <origin xyz="-0.005 0.0 -0.04499" rpy="${-PI/2} 0 0"/>
     </xacro:kobuki_caster>
-    <xacro:kobuki_lidar parent="base2_link">
+    <xacro:caster_gazebo prefix="back"/>
+                                                                          <!-- KOBUKI LIDAR -->
+    <!-- <xacro:kobuki_lidar parent="base2_link">
         <origin xyz="0.0 0.0 0.030" rpy="0 0 0"/>
     </xacro:kobuki_lidar>
+    <xacro:lidar_gazebo/> -->
+                                                                          <!-- KOBUKI IMU -->
     <xacro:kobuki_imu parent="base_link">
-        <origin xyz="0.056 0.062 0.0202" rpy="0 0 0"/>
+        <origin xyz="0.056 0.062 -0.03179" rpy="0 0 0"/>
     </xacro:kobuki_imu>
+    <xacro:imu_gazebo/>
+                                                                          <!-- KOBUKI RGBD CAMERA -->
+                                                      <!-- Simple representation of the realsense D415 depth camera -->
     <xacro:kobuki_camera parent="base_link">
-        <origin xyz="-0.0 0.0 0.11" rpy="0 0 0"/>
+        <origin xyz="0.165 0.0 0.05801" rpy="0 0 0"/>
     </xacro:kobuki_camera>
-    <!-- 1010 base2+lidar -->
-    <xacro:base1_gazebo/>
-    <xacro:base2_gazebo/>
-    <xacro:pc_gazebo/>
-    <xacro:hex_gazebo prefix="back_left"/>
-    <xacro:hex_gazebo prefix="back_right"/>
-    <xacro:hex_gazebo prefix="front_left"/>
-    <xacro:hex_gazebo prefix="front_right"/>
-    <xacro:caster_gazebo prefix="front"/>
-    <xacro:caster_gazebo prefix="back"/>
-    <xacro:wheel_gazebo prefix="right"/>
-    <xacro:wheel_gazebo prefix="left"/>
-    <xacro:lidar_gazebo/>
-    <xacro:imu_gazebo/>
-    <xacro:rgb_camera_gazebo/>
-    <xacro:depth_camera_gazebo/>
+    <!-- <xacro:rgb_camera_gazebo/>
+    <xacro:depth_camera_gazebo/> -->
+    <xacro:rgbd_camera/>
+                                                                          <!-- D1 ARM -->
+    <xacro:D1_robot parent="base2_link">
+        <origin xyz="0.0 0.0 0.0010" rpy="0 0 0"/>
+    </xacro:D1_robot>
+    <xacro:D1_gazebo/>
+                                                                          <!-- CONTROL -->
     <xacro:control_gazebo/>
 </robot>

File: src/kobuki_ros/kobuki_description/model/parts/kobuki_base.gazebo.xacro (robot description, xacro)
@@ -29,11 +29,11 @@
         <mu1 value="1.2" />
         <mu2 value="1.2" />
-        <material>Gazebo/DarkYellow</material>
+        <material>Gazebo/Red</material>
     </gazebo>
   </xacro:macro>
   <xacro:macro name="caster_gazebo" params="prefix">
     <gazebo reference="${prefix}_casters_link">
-        <mu1>0.0</mu1>
-        <mu2>0.0</mu2>
+        <mu1>0.0000001</mu1>
+        <mu2>0.0000001</mu2>
         <kp>1000000.0</kp>
         <kd>100.0</kd>

File: src/kobuki_ros/kobuki_description/model/parts/kobuki_base.xacro (robot description, xacro)
@@ -1,4 +1,5 @@
 <?xml version="1.0"?>
 <robot xmlns:xacro="https://www.ros.org/wiki/xacro">
+    <!-- <xacro:include filename="$(find kobuki_description)/model/common_properties.urdf.xacro"/> -->
     <xacro:include filename="$(find kobuki_description)/model/parts/kobuki_base.gazebo.xacro"/>
                                                                             <!-- KOBUKI BASE -->
@@ -14,5 +15,5 @@
                     <mesh filename="file://$(find kobuki_description)/meshes/main_body.dae" />
                 </geometry>
-                <origin xyz="0.001 0 0.05199" rpy="0 0 0"/>
+                <!-- <origin xyz="0.001 0 0.05199" rpy="0 0 0"/> -->
             </visual>
             <collision>
@@ -20,12 +21,17 @@
                     <cylinder length="0.10938" radius="0.178"/>
                 </geometry>
-            <origin xyz="0.0 0 0.05949" rpy="0 0 0"/>
+            <!-- <origin xyz="0.0 0 0.05949" rpy="0 0 0"/> -->
             </collision>
             <inertial>
                 <origin xyz="0.01 0 0"/>
-                <mass value="5.9"/>
-                <inertia ixx="0.019995" ixy="0.0" ixz="0.0"
-                        iyy="0.019995" iyz="0.0"
-                        izz="0.03675" />
+                <!-- kobuki mass = 2.4  pc mass = 1.46 -->
+                <!-- <mass value="3.86"/> -->
+                <mass value="2.4"/>
+                <inertia ixx="0.0001" ixy="0.0" ixz="0.0"
+                        iyy="0.0001" iyz="0.0"
+                        izz="0.0001" />
+                <!-- <inertia ixx="0.021403197" ixy="0.0" ixz="0.0"
+                        iyy="0.021403197" iyz="0.0"
+                        izz="0.0380208" /> -->
             </inertial>
         </link>
@@ -42,25 +48,25 @@
             <visual>
                 <geometry>
-                    <mesh filename="file://$(find kobuki_description)/meshes/stl/BASE2.stl" scale="0.001 0.001 0.001"/>
-                    <!-- <cylinder length="0.01" radius="0.15"/> -->
+                    <mesh filename="file://$(find kobuki_description)/meshes/stl/BASE2_scaled_rotated.stl"/>
                 </geometry>
-                <origin xyz="-0.0 -0.0 0.0" rpy="0 0 ${PI/2}"/>
+                <!-- <origin xyz="-0.0 -0.0 0.0" rpy="0 0 ${PI/2}"/> -->
+                <xacro:insert_block name="material_black"/>
             </visual>
             <collision>
                 <geometry>
-                    <mesh filename="file://$(find kobuki_description)/meshes/stl/BASE2.stl" scale="0.001 0.001 0.001"/>
+                    <mesh filename="file://$(find kobuki_description)/meshes/stl/BASE2_scaled_rotated.stl"/>
                     <!-- <cylinder length="0.01" radius="0.15"/> -->
                 </geometry>
-            <origin xyz="-0.0 -0.0 0.0" rpy="0 0 ${PI/2}"/>
+            <!-- <origin xyz="-0.0 -0.0 0.0" rpy="0 0 ${PI/2}"/> -->
             </collision>
             <inertial>
                 <origin xyz="0 0 0"/>
                 <mass value="0.840"/>
-                <!-- <inertia ixx="0.000000005" ixy="0.0" ixz="0.0"
-                        iyy="0.000000005" iyz="0.0"
-                        izz="0.00945" /> -->
-                <inertia ixx="0.004725" ixy="0.0" ixz="0.0"
-                        iyy="0.004725" iyz="0.0"
-                        izz="0.00945" />
+                <inertia ixx="0.00305872" ixy="0.0" ixz="0.0"
+                        iyy="0.00239157" iyz="0.0"
+                        izz="0.0054502" />
+                <!-- <inertia ixx="0.0001" ixy="0.0" ixz="0.0"
+                        iyy="0.0001" iyz="0.0"
+                        izz="0.0001" /> -->
             </inertial>
         </link>
@@ -76,23 +82,23 @@
             <visual>
                 <geometry>
-                    <mesh filename="file://$(find kobuki_description)/meshes/stl/kobuki_pc2.stl" scale="0.01 0.01 0.01"/>
-                    <!-- <cylinder length="0.01" radius="0.15"/> -->
+                    <mesh filename="file://$(find kobuki_description)/meshes/stl/kobuki_pc2_rotated.stl"/>
                 </geometry>
-                <origin xyz="-0.0 -0.0 0.0" rpy="0 0 0"/>
+                <xacro:insert_block name="material_dark_grey"/>
+                <!-- <origin xyz="-0.0 -0.0 0.0" rpy="0 0 ${PI}"/> -->
             </visual>
             <collision>
                 <geometry>
-                    <!-- <mesh filename="file://$(find kobuki_description)/meshes/stl/kobuki_pc2.stl" scale="0.01 0.01 0.01"/> -->
-                    <box size="0.20 0.20 0.075"/>
+                    <mesh filename="file://$(find kobuki_description)/meshes/stl/kobuki_pc2_rotated.stl"/>
+                    <!-- <box size="0.1778 0.1829 0.075"/> -->
                 </geometry>
-            <origin xyz="-0.0 -0.0 0.0" rpy="0 0 0"/>
+                <!-- <origin xyz="-0.0 -0.0 0.0" rpy="0 0 ${PI}"/> -->
             </collision>
-            <!-- <inertial>
+            <inertial>
                 <origin xyz="0 0 0"/>
-                <mass value="3.5"/>
-                <inertia ixx="0.0000007" ixy="0.0" ixz="0.0"
-                        iyy="0.0000007" iyz="0.0"
-                        izz="0.0000014" />
-            </inertial> -->
+                <mass value="1.46"/>
+                <inertia ixx="0.00359729" ixy="0.0" ixz="0.0"
+                        iyy="0.00414973" iyz="0.0"
+                        izz="0.00706535" />
+            </inertial>
         </link>
     </xacro:macro>
@@ -110,4 +116,5 @@
                 </geometry>
                 <origin xyz="0.0 0 0.0" rpy="0 0 0"/>
+                <xacro:insert_block name="material_red"/>
             </visual>
             <collision>

File: src/kobuki_ros/kobuki_description/model/sensors/imu/kobuki_imu.gazebo.xacro (robot description, xacro)
@@ -5,10 +5,9 @@
         <gravity>true</gravity>
         <sensor name="imu_sensor" type="imu">
-            <plugin filename="gz-sim-imu-system" name="gz::sim::systems::Imu">
-            </plugin>
             <always_on>true</always_on>
-            <update_rate>1</update_rate>
+            <update_rate>50</update_rate>
             <visualize>true</visualize>
             <topic>/imu</topic>
+            <gz_frame_id>imu_link</gz_frame_id>
             <imu>
                 <noise>
@@ -27,4 +26,5 @@
                         </accel>
                 </noise>
+                <frame_id>imu_link</frame_id>
             </imu>
         </sensor>

File: src/kobuki_ros/kobuki_description/model/sensors/imu/kobuki_imu.xacro (robot description, xacro)
@@ -14,6 +14,6 @@
                 <origin xyz="0 0 0" rpy="0 0 0"/>
                 <inertia ixx="0.0001" ixy="0" ixz="0"
-                        iyy="0.000001" iyz="0"
-                        izz="0.0001"/>
+                         iyy="0.000001" iyz="0"
+                         izz="0.0001"/>
             </inertial>
         </link>

File: src/kobuki_ros/kobuki_description/model/sensors/lidar/kobuki_lidar.gazebo.xacro (robot description, xacro)
@@ -6,12 +6,13 @@
         <selfCollide>false</selfCollide>
         <sensor name="gpu_lidar" type="gpu_lidar">
-            <plugin filename="gz-sim-sensors-system" name="gz::sim::systems::Sensors">
+            <pose> 0 0 0.0215 0 0 0 </pose>
+            <!-- <plugin filename="gz-sim-sensors-system" name="gz::sim::systems::Sensors">
                 <render_engine>ogre2</render_engine>
-            </plugin>
+            </plugin> -->
             <always_on>true</always_on>
             <update_rate>10</update_rate>
             <visualize>1</visualize>
             <gz_frame_id>lidar_link</gz_frame_id>
-            <topic>lidar</topic>
+            <topic>scan</topic>
             <lidar>
                 <scan>
@@ -19,6 +20,6 @@
                         <samples>800</samples>
                         <resolution>1</resolution>
-                        <min_angle>-3.1415926535897931</min_angle>
-                        <max_angle>3.1415926535897931</max_angle>
+                        <min_angle>${-PI}</min_angle>
+                        <max_angle>${PI}</max_angle>
                     </horizontal>
                     <vertical>
@@ -34,5 +35,5 @@
                     <resolution>0.01</resolution>
                 </range>
-                <frame_id>/lidar_link</frame_id>
+                <!-- <frame_id>/lidar_link</frame_id> -->
             </lidar>
         </sensor>

File: src/kobuki_ros/kobuki_description/model/sensors/lidar/kobuki_lidar.xacro (robot description, xacro)
@@ -10,16 +10,12 @@
         <link name="lidar_link">
             <visual>
-                <!-- <origin xyz="-0.0475 0.035 0.02" rpy="${PI/2} 0 0"/> -->
-                <origin xyz="-0.0 0.0 -0.0" rpy="0 0 0"/>
                 <geometry>
-                    <mesh filename="file://$(find kobuki_description)/meshes/stl/lidar2.stl" scale="0.01 0.01 0.01"/>
+                    <mesh filename="file://$(find kobuki_description)/meshes/stl/lidar2_rotated.stl"/>
                 </geometry>
             </visual>
             <collision>
                 <geometry>
-                    <mesh filename="file://$(find kobuki_description)/meshes/stl/lidar2.stl" scale="0.01 0.01 0.01"/>
+                    <mesh filename="file://$(find kobuki_description)/meshes/stl/lidar2_rotated.stl"/>
                 </geometry>
-                <!-- <origin rpy="${PI/2} 0 0" xyz="-0.0475 0.035 -0.0225"/> -->
-                <origin xyz="-0.0 0.0 -0.0" rpy="0 0 0"/>
             </collision>
             <inertial>

File: src/kobuki_ros/kobuki_description/model/wheels/kobuki_wheels.gazebo.xacro (robot description, xacro)
@@ -8,5 +8,5 @@
         <kd>100.0</kd>
         <minDepth>0.001</minDepth>
-        <maxVel>10.0</maxVel>
+        <maxVel>1.0</maxVel>
         <!-- <material>Gazebo/Yellow</material> -->
     </gazebo>
