Commit message: 14-07-25

File: src/kobuki_ros/kobuki_description/model/wheels/kobuki_wheels.xacro (robot description, xacro)
@@ -7,5 +7,5 @@
             <parent link="${parent}"/>
             <child link="${prefix}_wheel_link"/>
-            <limit effort="50000" velocity="20"/>
+            <limit effort="50000" velocity="${max_vel}"/>
             <dynamics damping="1.0" friction="1.0"/>
             <axis xyz="0 0 1"/>

Commit message: Add optical link for the camera

File: src/kobuki_ros/kobuki_description/model/camera/kobuki_camera.gazebo.xacro (robot description, xacro)
@@ -52,12 +52,12 @@
     <gazebo reference="camera_link">
         <sensor name="rgbd_camera" type="rgbd_camera">
-            <!-- <pose relative_to='camera_link'> 0 0 0 0 -0.174532925 0 </pose> -->
-            <pose relative_to='camera_link'> 0 0 0 0 0 0 </pose>
             <gz_frame_id>camera_link</gz_frame_id>
             <topic>rgbd_camera</topic>
             <always_on>1</always_on>
-            <update_rate>2</update_rate>
+            <update_rate>30</update_rate>
             <camera>
                 <horizontal_fov>1.134464014</horizontal_fov>
+                <optical_frame_id>camera_link_optical</optical_frame_id>
+                <!-- <camera_info_topic>camera/camera_info</camera_info_topic> -->
                 <image>
                     <width>320</width>
@@ -66,5 +66,5 @@
                 <clip>
                     <near>0.1</near>
-                    <far>5</far>
+                    <far>10</far>
                 </clip>
             </camera>

File: src/kobuki_ros/kobuki_description/model/camera/kobuki_camera.xacro (robot description, xacro)
@@ -14,5 +14,5 @@
                 </geometry>
                 <xacro:insert_block name="material_light_grey"/>
-                <origin xyz="0 0 0" rpy="0 ${PI/2} 0"/>
+                <!-- <origin xyz="0 0 0" rpy="0 ${PI/2} 0"/> -->
             </visual>
             <collision>
@@ -20,5 +20,5 @@
                     <mesh filename="file://$(find kobuki_description)/meshes/stl/d415s_rotated.stl" />
                 </geometry>
-                <origin xyz="0 0 0" rpy="0 ${PI/2} 0"/>
+                <!-- <origin xyz="0 0 0" rpy="0 ${PI/2} 0"/> -->
             </collision>
             <inertial>
@@ -29,3 +29,12 @@
         </link>
     </xacro:macro>
+    <xacro:macro name="kobuki_optical_camera" params="parent *joint_origin">
+        <joint name="camera__optical_joint" type="fixed">
+            <xacro:insert_block name="joint_origin"/>
+            <parent link="${parent}"/>
+            <child link="camera_link_optical"/>
+        </joint>
+        <link name="camera_link_optical">
+        </link>
+    </xacro:macro>
 </robot>

File: src/kobuki_ros/kobuki_description/model/kobuki_d1_sim.xacro (robot description, xacro)
@@ -75,4 +75,7 @@
         <origin xyz="0.165 0.0 0.05801" rpy="0 0 0"/>
     </xacro:kobuki_camera>
+    <xacro:kobuki_optical_camera parent="camera_link">
+        <origin xyz="0 0 0" rpy="-1.57 0 -1.57"/>
+    </xacro:kobuki_optical_camera>
     <!-- <xacro:rgb_camera_gazebo/>
     <xacro:depth_camera_gazebo/> -->

File: src/kobuki_ros/kobuki_description/model/kobuki_sim.xacro (robot description, xacro)
@@ -38,5 +38,5 @@
     </xacro:kobuki_hex>
     <xacro:hex_gazebo prefix="front_left"/>
-    <xacro:kobuki_hex parent="base_link" prefix="front_right">w
+    <xacro:kobuki_hex parent="base_link" prefix="front_right">
       <origin xyz="0.055 0.12 0.06901"/>
     </xacro:kobuki_hex>
@@ -74,4 +74,7 @@
         <origin xyz="0.165 0.0 0.05801" rpy="0 0 0"/>
     </xacro:kobuki_camera>
+    <xacro:kobuki_optical_camera parent="camera_link">
+        <origin xyz="0 0 0" rpy="-1.57 0 -1.57"/>
+    </xacro:kobuki_optical_camera>
     <!-- <xacro:rgb_camera_gazebo/>
     <xacro:depth_camera_gazebo/> -->
